File: pcb/CoCoQuadLink.brd (EAGLE design)
At the start: 97.8 x 66.7 mm, 80 parts, among them IC1 XC95144XLTQG100, IC10 MAX232, IC11 MAX232, IC13 ASE, IC14 SC16C752, IC2 AM29F040J, IC3 XC9572XLTQG100, IC4 65X51A, IC5 65X51A, IC8 MAX232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

Commit message: Refreshed PCB
Parts:
- removed IC14: SC16C752, nxp-jlb:LQFP48
- added C7.1: .1, rcl:C0402
- added IC6: ST16C550, texas-jlb:LQFP48
- added IC7: TL16C550, texas-jlb:LQFP48
Connections:
- removed net !IOR: IC1.68, IC14.19
- removed net !IOW: IC1.71, IC14.15
- new net IOR: IC1.68, IC6.20, IC7.20
- new net IOW: IC1.71, IC6.17, IC7.17
- new net N$33: IC6.12, IC6.5
- new net N$35: IC7.12, IC7.5
- new net OUT2_UART2: IC6.31
- new net OUT2_UART3: IC7.31
- net !UART_CTS2: now also IC6.38; no longer IC14.38
- net !UART_CTS3: now also IC7.38; no longer IC14.23
- net !UART_DCD2: now also IC6.40; no longer IC14.40
- net !UART_DCD3: now also IC7.40; no longer IC14.16
- net !UART_DSR2: now also IC6.39; no longer IC14.39
- net !UART_DSR3: now also IC7.39; no longer IC14.20
- net !UART_DTR2: now also IC6.33; no longer IC14.34
- net !UART_DTR3: now also IC7.33; no longer IC14.35
- net !UART_RTS2: now also IC6.32; no longer IC14.33
- net !UART_RTS3: now also IC7.32; no longer IC14.22
- net !UART_RXD3: now also IC7.7; no longer IC14.4
- net !UART_TXD3: now also IC7.8; no longer IC14.8
- net A0: now also IC6.28, IC7.28; no longer IC14.28
- net A1: now also IC6.27, IC7.27; no longer IC14.27
- net A2: now also IC6.26, IC7.26; no longer IC14.26
- net BD0: now also IC6.43, IC7.43; no longer IC14.44
- net BD1: now also IC6.44, IC7.44; no longer IC14.45
- net BD2: now also IC6.45, IC7.45; no longer IC14.46
- net BD3: now also IC6.46, IC7.46; no longer IC14.47
- net BD4: now also IC6.47, IC7.47; no longer IC14.48
- net BD5: now also IC6.2, IC7.2; no longer IC14.1
- net BD6: now also IC6.3, IC7.3; no longer IC14.2
- net BD7: now also IC6.4, IC7.4; no longer IC14.3
- net CE_UART2: now also IC6.10, IC6.9; no longer IC14.10
- net CE_UART3: now also IC7.10, IC7.9; no longer IC14.11
- net GND: now also C7.1.2, IC6.11, IC6.16, IC6.18, IC6.19, IC6.24, IC7.11, IC7.16, IC7.18, IC7.19, IC7.24; no longer IC14.17
- net INT_UART2: now also IC6.30; no longer IC14.30
- net INT_UART3: now also IC7.30; no longer IC14.29
- net OUT1_UART2: now also IC6.34; no longer IC14.32
- net OUT1_UART3: now also IC7.34; no longer IC14.9
- net RESET: now also IC6.35, IC7.35; no longer IC14.36
- net UART_CLK: now also IC6.14, IC7.14; no longer IC14.13
- net UART_RXD2: now also IC6.7; no longer IC14.5
- net UART_TXD2: now also IC6.8; no longer IC14.7
- net VCC: now also C7.1.1, IC6.41, IC6.42, IC7.41, IC7.42; no longer IC14.21, IC14.41, IC14.42
Routing:
- net IOR: track 0.00 -> 100.8 mm, vias 0 -> 3
- net IOW: track 0.00 -> 99.1 mm, vias 0 -> 3
- net !IOR: track 90.7 -> 0.00 mm, vias 2 -> 0
- net !IOW: track 90.4 -> 0.00 mm, vias 2 -> 0
- net !UART_DCD3: track 0.00 -> 80.7 mm
- net !UART_DSR3: track 0.00 -> 79.4 mm
- net !UART_CTS3: track 0.00 -> 78.1 mm
- net !UART_RTS3: track 0.00 -> 75.7 mm
- net A2: track 84.0 -> 153.6 mm, vias 2 -> 3
- net !UART_RXD3: track 0.00 -> 62.6 mm
- net !UART_TXD3: track 0.00 -> 61.9 mm
- net !UART_DTR3: track 37.2 -> 72.4 mm
- net INT_UART3: track 7.16 -> 31.2 mm, vias 0 -> 2
- net RESET: track 87.7 -> 105.4 mm, vias 2 -> 3
- net BD7: track 115.1 -> 127.7 mm
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