File: pcb/CoCoQuadLink.sch (EAGLE design)
At the start: 80 parts, among them IC1 XC95144XLTQG100, IC10 MAX232, IC11 MAX232, IC13 ASE, IC14 SC16C752, IC2 AM29F040J, IC3 XC9572XLTQG100, IC4 65X51A, IC5 65X51A, IC8 MAX232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

Commit message: Refreshed PCB
Parts:
- removed IC14: SC16C752, nxp-jlb:SC16C752
- added C7.1: .1, rcl:C-USC0402
- added IC6: ST16C550, texas-jlb:TLC550PT
- added IC7: TL16C550, texas-jlb:TLC550PT
Connections:
- removed net !IOR: IC1.68FB8MC11, IC14I.!IOR
- removed net !IOW: IC1.71FB8MC14, IC14I.!IOW
- new net IOR: IC1.68FB8MC11, IC6A.IOR, IC7A.IOR
- new net IOW: IC1.71FB8MC14, IC6A.IOW, IC7A.IOW
- new net N$33: IC6A.!BAUDOUT, IC6A.RCLK
- new net N$35: IC7A.!BAUDOUT, IC7A.RCLK
- new net OUT2_UART2: IC6A.!OUT2
- new net OUT2_UART3: IC7A.!OUT2
- net !UART_CTS2: now also IC6A.!CTS; no longer IC14A.!CTS
- net !UART_CTS3: now also IC7A.!CTS; no longer IC14B.!CTS
- net !UART_DCD2: now also IC6A.!DCD; no longer IC14A.!DCD
- net !UART_DCD3: now also IC7A.!DCD; no longer IC14B.!DCD
- net !UART_DSR2: now also IC6A.!DSR; no longer IC14A.!DSR
- net !UART_DSR3: now also IC7A.!DSR; no longer IC14B.!DSR
- net !UART_DTR2: now also IC6A.!DTR; no longer IC14A.!DTR
- net !UART_DTR3: now also IC7A.!DTR; no longer IC14B.!DTR
- net !UART_RTS2: now also IC6A.!RTS; no longer IC14A.!RTS
- net !UART_RTS3: now also IC7A.!RTS; no longer IC14B.!RTS
- net !UART_RXD3: now also IC7A.RXD; no longer IC14B.RXD
- net !UART_TXD3: now also IC7A.TXD; no longer IC14B.TXD
- net A0: now also IC6A.A0, IC7A.A0; no longer IC14I.A0
- net A1: now also IC6A.A1, IC7A.A1; no longer IC14I.A1
- net A2: now also IC6A.A2, IC7A.A2; no longer IC14I.A2
- net BD0: now also IC6A.D0, IC7A.D0; no longer IC14I.D0
- net BD1: now also IC6A.D1, IC7A.D1; no longer IC14I.D1
- net BD2: now also IC6A.D2, IC7A.D2; no longer IC14I.D2
- net BD3: now also IC6A.D3, IC7A.D3; no longer IC14I.D3
- net BD4: now also IC6A.D4, IC7A.D4; no longer IC14I.D4
- net BD5: now also IC6A.D5, IC7A.D5; no longer IC14I.D5
- net BD6: now also IC6A.D6, IC7A.D6; no longer IC14I.D6
- net BD7: now also IC6A.D7, IC7A.D7; no longer IC14I.D7
- net CE_UART2: now also IC6A.CS0, IC6A.CS1; no longer IC14I.!CSA
- net CE_UART3: now also IC7A.CS0, IC7A.CS1; no longer IC14I.!CSB
- net GND: now also C7.1.2, IC6A.!ADS, IC6A.!CS2, IC6A.!IOR, IC6A.!IOW, IC6P.GND, IC7A.!ADS, IC7A.!CS2, IC7A.!IOR, IC7A.!IOW, IC7P.GND; no longer IC14P.GND
- net INT_UART2: now also IC6A.INTRPT; no longer IC14A.INT
- net INT_UART3: now also IC7A.INTRPT; no longer IC14B.INT
- net OUT1_UART2: now also IC6A.!OUT1; no longer IC14A.!OUT
- net OUT1_UART3: now also IC7A.!OUT1; no longer IC14B.!OUT
- net RESET: now also IC6A.RESET, IC7A.RESET; no longer IC14I.RESET
- net UART_CLK: now also IC6A.XTAL1, IC7A.XTAL1; no longer IC14I.XTAL1
- net UART_RXD2: now also IC6A.RXD; no longer IC14A.RXD
- net UART_TXD2: now also IC6A.TXD; no longer IC14A.TXD
- net VCC: now also C7.1.1, IC6A.!RI, IC6P.VCC, IC7A.!RI, IC7P.VCC; no longer IC14A.!RI, IC14B.!RI, IC14P.VCC
Other:
- moved on the sheet: C4.1, C5.1, C6.1, IC4, IC4P, IC5, IC5P
